Commit message: Added simplified ardrone model, implemented IR sensor xacro

File: rotors_description/urdf/ardrone.xacro (robot description, xacro)
@@ -5,8 +5,10 @@
   <xacro:property name="rotor_velocity_slowdown_sim" value="10" />
   <xacro:property name="use_mesh_file" value="true" />
+  <xacro:property name="use_simplified_mesh_file" value="true" />
   <xacro:property name="mesh_file" value="package://rotors_description/meshes/ardrone.dae" />
+  <xacro:property name="simplified_mesh_file" value="package://rotors_description/meshes/ardrone_simplified.dae" />
   <xacro:property name="mass" value="1.5" /> <!-- [kg] -->
   <xacro:property name="body_width" value="0.3" /> <!-- [m] -->
-  <xacro:property name="body_height" value="0.16" /> <!-- [m] -->
+  <xacro:property name="body_height" value="0.08" /> <!-- [m] -->
   <xacro:property name="mass_rotor" value="0.005" /> <!-- [kg] -->
   <xacro:property name="arm_length" value="0.09" /> <!-- [m] -->

File: rotors_description/urdf/ardrone_base.xacro (robot description, xacro)
@@ -6,10 +6,13 @@
   <!-- Instantiate a controller. -->
   <xacro:controller_plugin_macro namespace="${namespace}" imu_sub_topic="imu" />
-  <xacro:if value="$(arg enable_mavlink_interface)">
-    <!-- Instantiate mavlink telemetry interface. -->
+  <!-- <xacro:if value="$(arg enable_mavlink_interface)">
     <xacro:default_mavlink_interface namespace="${namespace}" imu_sub_topic="imu" rotor_count="4" />
-  </xacro:if>
+  </xacro:if> -->
   <!-- Mount an ADIS16448 IMU. -->
   <xacro:default_imu namespace="${namespace}" parent_link="${namespace}/base_link" />
+  <!-- Mount an IR. -->
+    <xacro:default_ir namespace="${namespace}" parent_link="${namespace}/base_link">
+        <origin xyz="0 0 -0.005" rpy="0 1.57 0"/>
+    </xacro:default_ir>
   <xacro:if value="$(arg enable_ground_truth)">
     <xacro:ground_truth_imu_and_odometry namespace="${namespace}" parent_link="${namespace}/base_link" />
