Commit message: Added simplified ardrone model, implemented IR sensor xacro

File: rotors_description/urdf/component_snippets.xacro (robot description, xacro)
@@ -19,6 +19,5 @@
   <xacro:property name="pi" value="3.14159265359" />
   <!-- Macro to add logging to a bag file. -->
-  <xacro:macro name="bag_plugin_macro"
-    params="namespace bag_file rotor_velocity_slowdown_sim wait_to_record_bag">
+  <xacro:macro name="bag_plugin_macro" params="namespace bag_file rotor_velocity_slowdown_sim wait_to_record_bag">
     <gazebo>
       <plugin filename="librotors_gazebo_bag_plugin.so" name="rosbag">
@@ -28,11 +27,10 @@
         <frameId>${namespace}/base_link</frameId>
         <rotorVelocitySlowdownSim>${rotor_velocity_slowdown_sim}</rotorVelocitySlowdownSim>
-	<waitToRecordBag>${wait_to_record_bag}</waitToRecordBag>
+        <waitToRecordBag>${wait_to_record_bag}</waitToRecordBag>
       </plugin>
     </gazebo>
   </xacro:macro>
   <!-- Macro to add a camera. -->
-  <xacro:macro name="camera_macro"
-    params="namespace parent_link camera_suffix frame_rate
+  <xacro:macro name="camera_macro" params="namespace parent_link camera_suffix frame_rate
       horizontal_fov image_width image_height image_format min_distance
       max_distance noise_mean noise_stddev enable_visual *geometry *origin">
@@ -65,5 +63,5 @@
     </joint>
     <link name="${namespace}/camera_${camera_suffix}_optical_link" />
-    <joint name="${namespace}/camera_${camera_suffix}_optical_joint" type="fixed" >
+    <joint name="${namespace}/camera_${camera_suffix}_optical_joint" type="fixed">
       <origin xyz="0 0 0" rpy="${-pi/2} 0 ${-pi/2}" />
       <parent link="${namespace}/camera_${camera_suffix}_link" />
@@ -113,6 +111,5 @@
   <!-- Camera joint macro - just the joints, links, and collisions for a single
        camera. -->
-  <xacro:macro name="camera_joint_macro"
-    params="namespace parent_link camera_suffix enable_visual *origin *geometry" >
+  <xacro:macro name="camera_joint_macro" params="namespace parent_link camera_suffix enable_visual *origin *geometry">
     <link name="${namespace}/camera_${camera_suffix}_link">
       <collision>
@@ -144,8 +141,7 @@
   </xacro:macro>
   <!-- Camera sensor macro - just image parameters. -->
-  <xacro:macro name="camera_sensor_macro"
-    params="camera_suffix horizontal_fov image_width image_height
+  <xacro:macro name="camera_sensor_macro" params="camera_suffix horizontal_fov image_width image_height
       image_format min_distance max_distance noise_mean noise_stddev
-      baseline" >
+      baseline">
     <camera name="${camera_suffix}">
       <pose>0 ${-baseline} 0 0 0 0</pose>
@@ -171,6 +167,5 @@
   </xacro:macro>
   <!-- Macro to add a multicamera (stereo pair). -->
-  <xacro:macro name="stereo_camera_macro"
-    params="namespace camera_name parent_link frame_rate
+  <xacro:macro name="stereo_camera_macro" params="namespace camera_name parent_link frame_rate
       horizontal_fov image_width image_height image_format min_distance
       max_distance noise_mean noise_stddev enable_visual origin_offset_x
@@ -178,18 +173,14 @@
     <!-- These are parameters for the left camera link and then the right
         as well. -->
-    <xacro:camera_joint_macro namespace="${namespace}"
-      parent_link="${parent_link}"
-      camera_suffix="left" enable_visual="${enable_visual}">
+    <xacro:camera_joint_macro namespace="${namespace}" parent_link="${parent_link}" camera_suffix="left" enable_visual="${enable_visual}">
       <origin xyz="${origin_offset_x} ${baseline_y/2} ${origin_offset_z}" rpy="0 0 0" />
       <xacro:insert_block name="geometry" />
     </xacro:camera_joint_macro>
-    <xacro:camera_joint_macro namespace="${namespace}"
-      parent_link="${parent_link}"
-      camera_suffix="right" enable_visual="${enable_visual}">
+    <xacro:camera_joint_macro namespace="${namespace}" parent_link="${parent_link}" camera_suffix="right" enable_visual="${enable_visual}">
       <origin xyz="${origin_offset_x} ${-baseline_y/2} ${origin_offset_z}" rpy="0 0 0" />
       <xacro:insert_block name="geometry" />
     </xacro:camera_joint_macro>
     <link name="${namespace}/camera_left_optical_link" />
-    <joint name="${namespace}/camera_left_optical_joint" type="fixed" >
+    <joint name="${namespace}/camera_left_optical_joint" type="fixed">
       <origin xyz="0 0 0" rpy="${-pi/2} 0 ${-pi/2}" />
       <parent link="${namespace}/camera_left_link" />
@@ -201,17 +192,7 @@
         <update_rate>${frame_rate}</update_rate>
         <!-- Here we set up the individual cameras of the stereo head. -->
-        <xacro:camera_sensor_macro camera_suffix="left"
-            horizontal_fov="${horizontal_fov}" image_width="${image_width}"
-            image_height="${image_height}" image_format="${image_format}"
-            min_distance="${min_distance}" max_distance="${max_distance}"
-            noise_mean="${noise_mean}" noise_stddev="${noise_stddev}"
-            baseline="0">
+        <xacro:camera_sensor_macro camera_suffix="left" horizontal_fov="${horizontal_fov}" image_width="${image_width}" image_height="${image_height}" image_format="${image_format}" min_distance="${min_distance}" max_distance="${max_distance}" noise_mean="${noise_mean}" noise_stddev="${noise_stddev}" baseline="0">
         </xacro:camera_sensor_macro>
-        <xacro:camera_sensor_macro camera_suffix="right"
-            horizontal_fov="${horizontal_fov}" image_width="${image_width}"
-            image_height="${image_height}" image_format="${image_format}"
-            min_distance="${min_distance}" max_distance="${max_distance}"
-            noise_mean="${noise_mean}" noise_stddev="${noise_stddev}"
-            baseline="${baseline_y}">
+        <xacro:camera_sensor_macro camera_suffix="right" horizontal_fov="${horizontal_fov}" image_width="${image_width}" image_height="${image_height}" image_format="${image_format}" min_distance="${min_distance}" max_distance="${max_distance}" noise_mean="${noise_mean}" noise_stddev="${noise_stddev}" baseline="${baseline_y}">
         </xacro:camera_sensor_macro>
         <!-- Stereo controller, setting the transforms between the two cameras. -->
@@ -249,7 +230,5 @@
   <!-- ==================== ROS INTERFACE MACRO ====================== -->
   <!-- =============================================================== -->
-  <!-- <xacro:macro
-  		name="ros_interface_plugin_macro"
-  		params="namespace">
+  <!-- <xacro:macro name="ros_interface_plugin_macro" params="namespace">
     <gazebo>
       <plugin name="ros_interface_plugin" filename="librotors_gazebo_ros_interface_plugin.so">
@@ -261,6 +240,5 @@
   <!-- ================== MAVLINK INTERFACE MACRO ==================== -->
   <!-- =============================================================== -->
-  <xacro:macro name="mavlink_interface_macro"
-    params="namespace mavlink_sub_topic imu_sub_topic mavlink_pub_topic
+  <xacro:macro name="mavlink_interface_macro" params="namespace mavlink_sub_topic imu_sub_topic mavlink_pub_topic
       motors_speeds_pub_topic gps_update_freq rotor_count reference_magnetic_field_north
       reference_magnetic_field_east reference_magnetic_field_down reference_latitude
@@ -269,10 +247,10 @@
       <plugin name="mavlink_interface" filename="librotors_gazebo_mavlink_interface.so">
         <robotNamespace>${namespace}</robotNamespace>
-	<mavlinkControlSubTopic>${mavlink_sub_topic}</mavlinkControlSubTopic>
+        <mavlinkControlSubTopic>${mavlink_sub_topic}</mavlinkControlSubTopic>
         <imuSubTopic>${imu_sub_topic}</imuSubTopic>
         <mavlinkHilSensorPubTopic>${mavlink_pub_topic}</mavlinkHilSensorPubTopic>
-	<motorSpeedsPubTopic>${motors_speeds_pub_topic}</motorSpeedsPubTopic>
-	<gpsUpdateFreq>${gps_update_freq}</gpsUpdateFreq> <!-- Frequency of HIL GPS messages [Hz] -->
-	<rotorCount>${rotor_count}</rotorCount>
+        <motorSpeedsPubTopic>${motors_speeds_pub_topic}</motorSpeedsPubTopic>
+        <gpsUpdateFreq>${gps_update_freq}</gpsUpdateFreq>        <!-- Frequency of HIL GPS messages [Hz] -->
+        <rotorCount>${rotor_count}</rotorCount>
         <!-- [Gauss] Below are the North, East, and Down components of the Earth's magnetic field at the reference location.
              The default reference location is Zurich (lat=+47.3667degN, lon=+8.5500degE, h=+500m, WGS84).
@@ -282,13 +260,68 @@
         <referenceMagEast>${reference_magnetic_field_east}</referenceMagEast>
         <referenceMagDown>${reference_magnetic_field_down}</referenceMagDown>
-	<referenceLatitude>${reference_latitude}</referenceLatitude> <!-- the initial latitude [degrees [-90, 90]] -->
-        <referenceLongitude>${reference_longitude}</referenceLongitude> <!-- the initial longitude [degrees [-180, 180]] -->
-        <referenceAltitude>${reference_altitude}</referenceAltitude> <!-- the initial altitude [m] -->
-      </plugin>
+        <referenceLatitude>${reference_latitude}</referenceLatitude>        <!-- the initial latitude [degrees [-90, 90]] -->
+        <referenceLongitude>${reference_longitude}</referenceLongitude>        <!-- the initial longitude [degrees [-180, 180]] -->
+        <referenceAltitude>${reference_altitude}</referenceAltitude>        <!-- the initial altitude [m] -->
+      </plugin>
+    </gazebo>
+  </xacro:macro>
+  <!-- Macro to add an IR. -->
+  <xacro:macro name="ir_plugin_macro" params="parent_link namespace ir_suffix ir_topic mass_ir_sensor *inertia *origin">
+      <!-- IR joint -->
+    <joint name="${namespace}/ir${ir_suffix}_joint" type="fixed">
+      <xacro:insert_block name="origin" />
+      <parent link="${parent_link}"/>
+      <child link="${namespace}/base_ir${ir_suffix}_link"/>
+    </joint>
+    <!-- IR link -->
+    <link name="${namespace}/base_ir${ir_suffix}_link">
+      <inertial>
+        <mass value="${mass_ir_sensor}" />
+        <xacro:insert_block name="inertia" />
+        <origin xyz="0 0 0" rpy="0 0 0" />
+      </inertial>
+    </link>
+    <gazebo reference="${namespace}/base_ir${ir_suffix}_link">
+      <sensor type="ray" name="TeraRanger">
+        <pose>0 0 0 0 0 0</pose>
+        <visualize>true</visualize>
+        <update_rate>50</update_rate>
+        <ray>
+          <scan>
+            <horizontal>
+              <samples>10</samples>
+              <resolution>1</resolution>
+              <min_angle>-0.01</min_angle>
+              <max_angle>0.01</max_angle>
+            </horizontal>
+            <vertical>
+              <samples>10</samples>
+              <resolution>1</resolution>
+              <min_angle>-0.01</min_angle>
+              <max_angle>0.01</max_angle>
+            </vertical>
+          </scan>
+          <range>
+            <min>0.01</min>
+            <max>2</max>
+            <resolution>0.01</resolution>
+          </range>
+        </ray>
+        <plugin filename="libgazebo_ros_range.so" name="gazebo_ros${ir_suffix}_range">
+          <robotNamespace>${namespace}</robotNamespace>
+          <gaussianNoise>0.001</gaussianNoise>
+          <alwaysOn>true</alwaysOn>
+          <updateRate>50</updateRate>
+          <topicName>${ir_topic}</topicName>
+          <!-- <frameName>${namespace}/base_ir${ir_suffix}_link</frameName> -->
+          <frameName>${namespace}/base_ir${ir_suffix}_link</frameName>
+          <radiation>INFRARED</radiation>
+          <fov>0.2967</fov>
+        </plugin>
+      </sensor>
     </gazebo>
   </xacro:macro>
   <!-- Macro to add an IMU. -->
-  <xacro:macro name="imu_plugin_macro"
-    params="namespace imu_suffix parent_link imu_topic
+  <xacro:macro name="imu_plugin_macro" params="namespace imu_suffix parent_link imu_topic
       mass_imu_sensor gyroscope_noise_density gyroscope_random_walk
       gyroscope_bias_correlation_time gyroscope_turn_on_bias_sigma
@@ -300,5 +333,6 @@
       <inertial>
         <xacro:insert_block name="inertia" />
-        <mass value="${mass_imu_sensor}" />  <!-- [kg] -->
+        <mass value="${mass_imu_sensor}" />
+        <!-- [kg] -->
         <origin xyz="0 0 0" rpy="0 0 0" />
       </inertial>
@@ -313,23 +347,22 @@
     <gazebo>
       <plugin filename="librotors_gazebo_imu_plugin.so" name="rotors_gazebo_imu${imu_suffix}_plugin">
-      <!-- A good description of the IMU parameters can be found in the kalibr documentation:
+        <!-- A good description of the IMU parameters can be found in the kalibr documentation:
            https://github.com/ethz-asl/kalibr/wiki/IMU-Noise-Model-and-Intrinsics -->
-        <robotNamespace>${namespace}</robotNamespace> <!-- (string, required): ros namespace in which the messages are published -->
-        <linkName>${namespace}/imu${imu_suffix}_link</linkName> <!-- (string, required): name of the body which holds the IMU sensor -->
-        <imuTopic>${imu_topic}</imuTopic> <!-- (string): name of the sensor output topic and prefix of service names (defaults to imu) -->
-        <gyroscopeNoiseDensity>${gyroscope_noise_density}</gyroscopeNoiseDensity> <!-- Gyroscope noise density (two-sided spectrum) [rad/s/sqrt(Hz)] -->
-        <gyroscopeRandomWalk>${gyroscope_random_walk}</gyroscopeRandomWalk> <!-- Gyroscope bias random walk [rad/s/s/sqrt(Hz)] -->
-        <gyroscopeBiasCorrelationTime>${gyroscope_bias_correlation_time}</gyroscopeBiasCorrelationTime> <!-- Gyroscope bias correlation time constant [s] -->
-        <gyroscopeTurnOnBiasSigma>${gyroscope_turn_on_bias_sigma}</gyroscopeTurnOnBiasSigma> <!-- Gyroscope turn on bias standard deviation [rad/s] -->
-        <accelerometerNoiseDensity>${accelerometer_noise_density}</accelerometerNoiseDensity> <!-- Accelerometer noise density (two-sided spectrum) [m/s^2/sqrt(Hz)] -->
-        <accelerometerRandomWalk>${accelerometer_random_walk}</accelerometerRandomWalk> <!-- Accelerometer bias random walk. [m/s^2/s/sqrt(Hz)] -->
-        <accelerometerBiasCorrelationTime>${accelerometer_bias_correlation_time}</accelerometerBiasCorrelationTime> <!-- Accelerometer bias correlation time constant [s] -->
-        <accelerometerTurnOnBiasSigma>${accelerometer_turn_on_bias_sigma}</accelerometerTurnOnBiasSigma> <!-- Accelerometer turn on bias standard deviation [m/s^2] -->
+        <robotNamespace>${namespace}</robotNamespace>        <!-- (string, required): ros namespace in which the messages are published -->
+        <linkName>${namespace}/imu${imu_suffix}_link</linkName>        <!-- (string, required): name of the body which holds the IMU sensor -->
+        <imuTopic>${imu_topic}</imuTopic>        <!-- (string): name of the sensor output topic and prefix of service names (defaults to imu) -->
+        <gyroscopeNoiseDensity>${gyroscope_noise_density}</gyroscopeNoiseDensity>        <!-- Gyroscope noise density (two-sided spectrum) [rad/s/sqrt(Hz)] -->
+        <gyroscopeRandomWalk>${gyroscope_random_walk}</gyroscopeRandomWalk>        <!-- Gyroscope bias random walk [rad/s/s/sqrt(Hz)] -->
+        <gyroscopeBiasCorrelationTime>${gyroscope_bias_correlation_time}</gyroscopeBiasCorrelationTime>        <!-- Gyroscope bias correlation time constant [s] -->
+        <gyroscopeTurnOnBiasSigma>${gyroscope_turn_on_bias_sigma}</gyroscopeTurnOnBiasSigma>        <!-- Gyroscope turn on bias standard deviation [rad/s] -->
+        <accelerometerNoiseDensity>${accelerometer_noise_density}</accelerometerNoiseDensity>        <!-- Accelerometer noise density (two-sided spectrum) [m/s^2/sqrt(Hz)] -->
+        <accelerometerRandomWalk>${accelerometer_random_walk}</accelerometerRandomWalk>        <!-- Accelerometer bias random walk. [m/s^2/s/sqrt(Hz)] -->
+        <accelerometerBiasCorrelationTime>${accelerometer_bias_correlation_time}</accelerometerBiasCorrelationTime>        <!-- Accelerometer bias correlation time constant [s] -->
+        <accelerometerTurnOnBiasSigma>${accelerometer_turn_on_bias_sigma}</accelerometerTurnOnBiasSigma>        <!-- Accelerometer turn on bias standard deviation [m/s^2] -->
       </plugin>
     </gazebo>
   </xacro:macro>
   <!-- Macro to add a generic odometry sensor. -->
-  <xacro:macro name="odometry_plugin_macro"
-    params="
+  <xacro:macro name="odometry_plugin_macro" params="
       namespace odometry_sensor_suffix parent_link pose_topic pose_with_covariance_topic
       position_topic transform_topic odometry_topic parent_frame_id child_frame_id
@@ -344,5 +377,6 @@
       <inertial>
         <xacro:insert_block name="inertia" />
-        <mass value="${mass_odometry_sensor}" />  <!-- [kg] -->
+        <mass value="${mass_odometry_sensor}" />
+        <!-- [kg] -->
       </inertial>
     </link>
@@ -363,20 +397,20 @@
         <transformTopic>${transform_topic}</transformTopic>
         <odometryTopic>${odometry_topic}</odometryTopic>
-        <parentFrameId>${parent_frame_id}</parentFrameId> <!-- Use the scoped link name here. e.g. Model::link. -->
+        <parentFrameId>${parent_frame_id}</parentFrameId>        <!-- Use the scoped link name here. e.g. Model::link. -->
         <childFrameId>${child_frame_id}</childFrameId>
-        <measurementDivisor>${measurement_divisor}</measurementDivisor> <!-- only every (seq % measurementDivisor) == 0 measurement is published [int] -->
-        <measurementDelay>${measurement_delay}</measurementDelay> <!-- time that measurement gets held back before it's published in [simulation cycles (int)] -->
-        <unknownDelay>${unknown_delay}</unknownDelay> <!-- additional delay, that just gets added to the timestamp [s] -->
-        <noiseNormalPosition>${noise_normal_position}</noiseNormalPosition> <!-- standard deviation of additive white gaussian noise [m] -->
-        <noiseNormalQuaternion>${noise_normal_quaternion}</noiseNormalQuaternion> <!-- standard deviation white gaussian noise [rad]: q_m = q*quaternionFromSmallAngleApproximation(noiseNormalQ) -->
-        <noiseNormalLinearVelocity>${noise_normal_linear_velocity}</noiseNormalLinearVelocity> <!-- standard deviation of additive white gaussian noise [m/s] -->
-        <noiseNormalAngularVelocity>${noise_normal_angular_velocity}</noiseNormalAngularVelocity> <!-- standard deviation of additive white gaussian noise [rad/s] -->
-        <noiseUniformPosition>${noise_uniform_position}</noiseUniformPosition> <!-- symmetric bounds of uniform noise [m] -->
-        <noiseUniformQuaternion>${noise_uniform_quaternion}</noiseUniformQuaternion> <!-- symmetric bounds of uniform noise [rad], computation see above -->
-        <noiseUniformLinearVelocity>${noise_uniform_linear_velocity}</noiseUniformLinearVelocity> <!-- symmetric bounds of uniform noise [m/s] -->
-        <noiseUniformAngularVelocity>${noise_uniform_angular_velocity}</noiseUniformAngularVelocity> <!-- symmetric bounds of uniform noise [rad/s] -->
+        <measurementDivisor>${measurement_divisor}</measurementDivisor>        <!-- only every (seq % measurementDivisor) == 0 measurement is published [int] -->
+        <measurementDelay>${measurement_delay}</measurementDelay>        <!-- time that measurement gets held back before it's published in [simulation cycles (int)] -->
+        <unknownDelay>${unknown_delay}</unknownDelay>        <!-- additional delay, that just gets added to the timestamp [s] -->
+        <noiseNormalPosition>${noise_normal_position}</noiseNormalPosition>        <!-- standard deviation of additive white gaussian noise [m] -->
+        <noiseNormalQuaternion>${noise_normal_quaternion}</noiseNormalQuaternion>        <!-- standard deviation white gaussian noise [rad]: q_m = q*quaternionFromSmallAngleApproximation(noiseNormalQ) -->
+        <noiseNormalLinearVelocity>${noise_normal_linear_velocity}</noiseNormalLinearVelocity>        <!-- standard deviation of additive white gaussian noise [m/s] -->
+        <noiseNormalAngularVelocity>${noise_normal_angular_velocity}</noiseNormalAngularVelocity>        <!-- standard deviation of additive white gaussian noise [rad/s] -->
+        <noiseUniformPosition>${noise_uniform_position}</noiseUniformPosition>        <!-- symmetric bounds of uniform noise [m] -->
+        <noiseUniformQuaternion>${noise_uniform_quaternion}</noiseUniformQuaternion>        <!-- symmetric bounds of uniform noise [rad], computation see above -->
+        <noiseUniformLinearVelocity>${noise_uniform_linear_velocity}</noiseUniformLinearVelocity>        <!-- symmetric bounds of uniform noise [m/s] -->
+        <noiseUniformAngularVelocity>${noise_uniform_angular_velocity}</noiseUniformAngularVelocity>        <!-- symmetric bounds of uniform noise [rad/s] -->
         <xacro:if value="${enable_odometry_map}">
-          <covarianceImage>package://rotors_gazebo/resource/${odometry_map}</covarianceImage> <!-- a bitmap image describing where the sensor works (white), and where not (black) -->
-          <covarianceImageScale>${image_scale}</covarianceImageScale> <!-- the scale of the image in the gazebo world, if set to 1.0, 1 pixel in the image corresponds to 1 meter in the world -->
+          <covarianceImage>package://rotors_gazebo/resource/${odometry_map}</covarianceImage>          <!-- a bitmap image describing where the sensor works (white), and where not (black) -->
+          <covarianceImageScale>${image_scale}</covarianceImageScale>          <!-- the scale of the image in the gazebo world, if set to 1.0, 1 pixel in the image corresponds to 1 meter in the world -->
         </xacro:if>
       </plugin>
@@ -384,6 +418,5 @@
   </xacro:macro>
   <!-- Macro to add a GPS sensor. -->
-  <xacro:macro name="gps_plugin_macro"
-    params="namespace gps_suffix parent_link gps_topic ground_speed_topic
+  <xacro:macro name="gps_plugin_macro" params="namespace gps_suffix parent_link gps_topic ground_speed_topic
       mass_gps_sensor horizontal_pos_std_dev vertical_pos_std_dev
       horizontal_vel_std_dev vertical_vel_std_dev *inertia *origin">
@@ -392,5 +425,6 @@
       <inertial>
         <xacro:insert_block name="inertia" />
-        <mass value="${mass_gps_sensor}" />  <!-- [kg] -->
+        <mass value="${mass_gps_sensor}" />
+        <!-- [kg] -->
         <origin xyz="0 0 0" rpy="0 0 0" />
       </inertial>
@@ -448,12 +482,12 @@
         </gps>
         <plugin filename="librotors_gazebo_gps_plugin.so" name="rotors_gazebo_gps${gps_suffix}_plugin">
-          <robotNamespace>${namespace}</robotNamespace> <!-- (string, required): ros namespace in which the messages are published -->
-          <linkName>${namespace}/gps${gps_suffix}_link</linkName> <!-- (string, required): name of the body which holds the GPS sensor -->
-          <gpsTopic>${gps_topic}</gpsTopic> <!-- (string): name of the sensor output topic and prefix of service names (defaults to 'gps') -->
-          <groundSpeedTopic>${ground_speed_topic}</groundSpeedTopic> <!-- (string): name of the ground speed output topic (defaults to 'ground_speed') -->
-          <horPosStdDev>${horizontal_pos_std_dev}</horPosStdDev> <!-- standard deviation for horizontal position noise [m] -->
-          <verPosStdDev>${vertical_pos_std_dev}</verPosStdDev> <!-- standard deviation for vertical position noise [m] -->
-          <horVelStdDev>${horizontal_vel_std_dev}</horVelStdDev> <!-- standard deviation for horizontal speed noise [m/s] -->
-          <verVelStdDev>${vertical_vel_std_dev}</verVelStdDev> <!-- standard deviation for vertical speed noise [m/s] -->
+          <robotNamespace>${namespace}</robotNamespace>          <!-- (string, required): ros namespace in which the messages are published -->
+          <linkName>${namespace}/gps${gps_suffix}_link</linkName>          <!-- (string, required): name of the body which holds the GPS sensor -->
+          <gpsTopic>${gps_topic}</gpsTopic>          <!-- (string): name of the sensor output topic and prefix of service names (defaults to 'gps') -->
+          <groundSpeedTopic>${ground_speed_topic}</groundSpeedTopic>          <!-- (string): name of the ground speed output topic (defaults to 'ground_speed') -->
+          <horPosStdDev>${horizontal_pos_std_dev}</horPosStdDev>          <!-- standard deviation for horizontal position noise [m] -->
+          <verPosStdDev>${vertical_pos_std_dev}</verPosStdDev>          <!-- standard deviation for vertical position noise [m] -->
+          <horVelStdDev>${horizontal_vel_std_dev}</horVelStdDev>          <!-- standard deviation for horizontal speed noise [m/s] -->
+          <verVelStdDev>${vertical_vel_std_dev}</verVelStdDev>          <!-- standard deviation for vertical speed noise [m/s] -->
         </plugin>
       </sensor>
@@ -461,6 +495,5 @@
   </xacro:macro>
   <!-- Macro to add a magnetometer. -->
-  <xacro:macro name="magnetometer_plugin_macro"
-    params="namespace magnetometer_suffix parent_link magnetometer_topic
+  <xacro:macro name="magnetometer_plugin_macro" params="namespace magnetometer_suffix parent_link magnetometer_topic
       mass_magnetometer_sensor ref_mag_north ref_mag_east ref_mag_down
       noise_normal noise_uniform_initial_bias *inertia *origin">
@@ -469,5 +502,6 @@
       <inertial>
         <xacro:insert_block name="inertia" />
-        <mass value="${mass_magnetometer_sensor}" />  <!-- [kg] -->
+        <mass value="${mass_magnetometer_sensor}" />
+        <!-- [kg] -->
         <origin xyz="0 0 0" rpy="0 0 0" />
       </inertial>
@@ -482,7 +516,7 @@
     <gazebo>
       <plugin filename="librotors_gazebo_magnetometer_plugin.so" name="rotors_gazebo_magnetometer${magnetometer_suffix}_plugin">
-        <robotNamespace>${namespace}</robotNamespace> <!-- (string, required): ros namespace in which the messages are published -->
-        <linkName>${namespace}/magnetometer${magnetometer_suffix}_link</linkName> <!-- (string, required): name of the body which holds the magnetometer -->
-        <magnetometerTopic>${magnetometer_topic}</magnetometerTopic> <!-- (string): name of the sensor output topic and prefix of service names (defaults to 'magnetic_field') -->
+        <robotNamespace>${namespace}</robotNamespace>        <!-- (string, required): ros namespace in which the messages are published -->
+        <linkName>${namespace}/magnetometer${magnetometer_suffix}_link</linkName>        <!-- (string, required): name of the body which holds the magnetometer -->
+        <magnetometerTopic>${magnetometer_topic}</magnetometerTopic>        <!-- (string): name of the sensor output topic and prefix of service names (defaults to 'magnetic_field') -->
         <!-- [Tesla] Below is the reference Earth's magnetic field at the reference location in NED frame.
              The default reference location is Zurich (lat=+47.3667degN, lon=+8.5500degE, h=+500m, WGS84).
@@ -492,12 +526,11 @@
         <refMagEast>${ref_mag_east}</refMagEast>
         <refMagDown>${ref_mag_down}</refMagDown>
-        <noiseNormal>${noise_normal}</noiseNormal> <!-- standard deviation of additive white gaussian noise [Tesla] -->
-        <noiseUniformInitialBias>${noise_uniform_initial_bias}</noiseUniformInitialBias> <!-- symmetric bounds of uniform noise for initial sensor bias [Tesla] -->
+        <noiseNormal>${noise_normal}</noiseNormal>        <!-- standard deviation of additive white gaussian noise [Tesla] -->
+        <noiseUniformInitialBias>${noise_uniform_initial_bias}</noiseUniformInitialBias>        <!-- symmetric bounds of uniform noise for initial sensor bias [Tesla] -->
       </plugin>
     </gazebo>
   </xacro:macro>
   <!-- Macro to add an air pressure sensor. -->
-  <xacro:macro name="pressure_sensor_plugin_macro"
-    params="namespace pressure_sensor_suffix parent_link pressure_topic
+  <xacro:macro name="pressure_sensor_plugin_macro" params="namespace pressure_sensor_suffix parent_link pressure_topic
       mass_pressure_sensor reference_altitude pressure_variance *inertia
       *origin">
@@ -506,5 +539,6 @@
       <inertial>
         <xacro:insert_block name="inertia" />
-        <mass value="${mass_pressure_sensor}" />  <!-- [kg] -->
+        <mass value="${mass_pressure_sensor}" />
+        <!-- [kg] -->
         <origin xyz="0 0 0" rpy="0 0 0" />
       </inertial>
@@ -519,15 +553,14 @@
     <gazebo>
       <plugin filename="librotors_gazebo_pressure_plugin.so" name="rotors_gazebo_pressure_sensor${pressure_sensor_suffix}_plugin">
-        <robotNamespace>${namespace}</robotNamespace> <!-- (string, required): ros namespace in which the messages are published -->
-        <linkName>${namespace}/pressure_sensor${pressure_sensor_suffix}_link</linkName> <!-- (string, required): name of the body which holds the pressure sensor -->
-        <pressureTopic>${pressure_topic}</pressureTopic> <!-- (string): name of the sensor output topic and prefix of service names (defaults to 'air_pressure') -->
-        <referenceAltitude>${reference_altitude}</referenceAltitude> <!-- the initial altitude [m] -->
-        <pressureVariance>${pressure_variance}</pressureVariance> <!-- the air pressure variance [Pa^2] -->
+        <robotNamespace>${namespace}</robotNamespace>        <!-- (string, required): ros namespace in which the messages are published -->
+        <linkName>${namespace}/pressure_sensor${pressure_sensor_suffix}_link</linkName>        <!-- (string, required): name of the body which holds the pressure sensor -->
+        <pressureTopic>${pressure_topic}</pressureTopic>        <!-- (string): name of the sensor output topic and prefix of service names (defaults to 'air_pressure') -->
+        <referenceAltitude>${reference_altitude}</referenceAltitude>        <!-- the initial altitude [m] -->
+        <pressureVariance>${pressure_variance}</pressureVariance>        <!-- the air pressure variance [Pa^2] -->
       </plugin>
     </gazebo>
   </xacro:macro>
   <!-- Macro to add the wind plugin. -->
-  <xacro:macro name="wind_plugin_macro"
-    params="namespace xyz_offset wind_direction wind_force_mean
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