Commit message: Added simplified ardrone model, implemented IR sensor xacro

File: rotors_description/urdf/multirotor_base.xacro (robot description, xacro)
@@ -19,7 +19,5 @@
   <!-- Macro for the inertia of a box -->
   <xacro:macro name="box_inertia" params="x y z mass">
-    <inertia ixx="${0.0833333 * mass * (y*y + z*z)}" ixy="0.0" ixz="0.0"
-      iyy="${0.0833333 * mass * (x*x + z*z)}" iyz="0.0"
-      izz="${0.0833333 * mass * (x*x + y*y)}" />
+    <inertia ixx="${0.0833333 * mass * (y*y + z*z)}" ixy="0.0" ixz="0.0" iyy="${0.0833333 * mass * (x*x + z*z)}" iyz="0.0" izz="${0.0833333 * mass * (x*x + y*y)}" />
   </xacro:macro>
   <!-- Macro for the inertial properties of a box -->
@@ -32,6 +30,5 @@
   </xacro:macro>
   <!-- Main multirotor link -->
-  <xacro:macro name="multirotor_base_macro"
-    params="robot_namespace mass body_width body_height use_mesh_file mesh_file *inertia">
+  <xacro:macro name="multirotor_base_macro" params="robot_namespace mass body_width body_height use_mesh_file mesh_file *inertia">
     <link name="${robot_namespace}/base_link"></link>
     <joint name="${robot_namespace}/base_joint" type="fixed">
@@ -42,5 +39,6 @@
     <link name="${robot_namespace}/base_link_inertia">
       <inertial>
-        <mass value="${mass}" />  <!-- [kg] -->
+        <mass value="${mass}" />
+        <!-- [kg] -->
         <origin xyz="0 0 0" />
         <xacro:insert_block name="inertia" />
@@ -53,5 +51,6 @@
           </xacro:if>
           <xacro:unless value="${use_mesh_file}">
-            <box size="${body_width} ${body_width} ${body_height}"/> <!-- [m] [m] [m] -->
+            <box size="${body_width} ${body_width} ${body_height}"/>
+            <!-- [m] [m] [m] -->
           </xacro:unless>
         </geometry>
@@ -60,6 +59,14 @@
         <origin xyz="0 0 0" rpy="0 0 0" />
         <geometry>
-          <box size="${body_width} ${body_width} ${body_height}" /> <!-- [m] [m] [m] -->
+          <xacro:if value="${use_simplified_mesh_file}">
+            <mesh filename="${simplified_mesh_file}" scale="1 1 1" />
+          </xacro:if>
+          <xacro:unless value="${use_simplified_mesh_file}">
+            <box size="${body_width} ${body_width} ${body_height}"/> <!-- [m] [m] [m] -->
+          </xacro:unless>
         </geometry>
+        <!-- <geometry>
+          <box size="${body_width} ${body_width} ${body_height}" />
+        </geometry> -->
       </collision>
     </link>
@@ -74,6 +81,5 @@
   </xacro:macro>
   <!-- Rotor joint and link -->
-  <xacro:macro name="vertical_rotor"
-    params="robot_namespace suffix direction motor_constant moment_constant parent mass_rotor radius_rotor time_constant_up time_constant_down max_rot_velocity motor_number rotor_drag_coefficient rolling_moment_coefficient color use_own_mesh mesh *origin *inertia">
+  <xacro:macro name="vertical_rotor" params="robot_namespace suffix direction motor_constant moment_constant parent mass_rotor radius_rotor time_constant_up time_constant_down max_rot_velocity motor_number rotor_drag_coefficient rolling_moment_coefficient color use_own_mesh mesh *origin *inertia">
     <joint name="${robot_namespace}/rotor_${motor_number}_joint" type="continuous">
       <xacro:insert_block name="origin" />
@@ -86,17 +92,17 @@
     <link name="${robot_namespace}/rotor_${motor_number}">
       <inertial>
-        <mass value="${mass_rotor}" /> <!-- [kg] -->
+        <mass value="${mass_rotor}" />
+        <!-- [kg] -->
         <xacro:insert_block name="inertia" />
       </inertial>
       <visual>
         <geometry>
-          <!-- <cylinder length="0.005" radius="${radius_rotor}"/> --> <!-- [m] -->
+          <!-- <cylinder length="0.005" radius="${radius_rotor}"/> -->          <!-- [m] -->
           <xacro:if value="${use_own_mesh}">
-            <mesh filename="${mesh}"
-              scale="1 1 1" />
+            <mesh filename="${mesh}" scale="1 1 1" />
           </xacro:if>
           <xacro:unless value="${use_own_mesh}">
-            <mesh filename="package://rotors_description/meshes/propeller_${direction}.dae"
-              scale="${radius_rotor} ${radius_rotor} ${radius_rotor}" /> <!-- The propeller meshes have a radius of 1m -->
+            <mesh filename="package://rotors_description/meshes/propeller_${direction}.dae" scale="${radius_rotor} ${radius_rotor} ${radius_rotor}" />
+            <!-- The propeller meshes have a radius of 1m -->
             <!-- <box size="${2*radius_rotor} 0.01 0.005"/> -->
           </xacro:unless>
@@ -105,5 +111,6 @@
       <collision>
         <geometry>
-          <cylinder length="0.005" radius="${radius_rotor}" /> <!-- [m] -->
+          <cylinder length="0.005" radius="${radius_rotor}" />
+          <!-- [m] -->
         </geometry>
       </collision>

Commit message: Flying boxes

File: rotors_description/urdf/ardrone.xacro (robot description, xacro)
@@ -4,5 +4,5 @@
   <xacro:property name="namespace" value="$(arg namespace)" />
   <xacro:property name="rotor_velocity_slowdown_sim" value="10" />
-  <xacro:property name="use_mesh_file" value="true" />
+  <xacro:property name="use_mesh_file" value="false" />
   <xacro:property name="use_simplified_mesh_file" value="true" />
   <xacro:property name="mesh_file" value="package://rotors_description/meshes/ardrone.dae" />

Commit message: Flying boxes are dead

File: rotors_description/urdf/ardrone.xacro (robot description, xacro)
@@ -4,5 +4,5 @@
   <xacro:property name="namespace" value="$(arg namespace)" />
   <xacro:property name="rotor_velocity_slowdown_sim" value="10" />
-  <xacro:property name="use_mesh_file" value="false" />
+  <xacro:property name="use_mesh_file" value="true" />
   <xacro:property name="use_simplified_mesh_file" value="true" />
   <xacro:property name="mesh_file" value="package://rotors_description/meshes/ardrone.dae" />
